File: PCB/Manette_JM/Manette_JM.kicad_pcb (KiCad board)
At the start: 2 copper layers, 33 parts, among them J1 Jack 1, J10 Bouton 2, J11 Bouton 3, J12 Bouton 4, J13 DEL PWR, J14 Joystick 0, J15 Jack 7, J16 Jack 8, J2 Jack 3, J3 Jack 4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

Commit message: PCB upgrade
Parts:
- added J17: Bouton3, Connector_PinHeader_2.54mm:PinHeader_1x02_P2.54mm_Vertical, F.Cu at (156.8, 92.2)
- added J18: Bouton4, Connector_PinHeader_2.54mm:PinHeader_1x02_P2.54mm_Vertical, F.Cu at (163.5, 92.2)
- added J19: Bouton5, Connector_PinHeader_2.54mm:PinHeader_1x02_P2.54mm_Vertical, F.Cu at (170.2, 92.3)
- added J20: DEL PWR, Connector_PinHeader_2.54mm:PinHeader_1x02_P2.54mm_Vertical, F.Cu at (170.2, 80.8)
- added J21: Joystick 0, Connector_PinHeader_2.54mm:PinHeader_1x04_P2.54mm_Vertical, F.Cu at (170.5, 54.5)
- added R16: 10K, Resistor_SMD:R_0805_2012Metric_Pad1.20x1.40mm_HandSolder, F.Cu at (150.0, 98.0)
- added R17: 10K, Resistor_SMD:R_0805_2012Metric_Pad1.20x1.40mm_HandSolder, F.Cu at (156.8, 98.0)
- added R18: 10K, Resistor_SMD:R_0805_2012Metric_Pad1.20x1.40mm_HandSolder, F.Cu at (163.5, 98.0)
- added R19: 10K, Resistor_SMD:R_0805_2012Metric_Pad1.20x1.40mm_HandSolder, F.Cu at (170.2, 98.0)
- added R20: 1.1K, Resistor_SMD:R_0805_2012Metric_Pad1.20x1.40mm_HandSolder, F.Cu at (170.2, 73.0)
- J10: value Bouton 2 -> Jack 10
- J11: value Bouton 3 -> Jack 11
- J12: value Bouton 4 -> Jack 12
- J13: value DEL PWR -> Jack 13
- J14: value Joystick 0 -> Jack 14; footprint Connector_PinHeader_2.54mm:PinHeader_1x04_P2.54mm_Vertical -> Connector_PinHeader_2.54mm:PinHeader_1x02_P2.54mm_Vertical
- J15: value Jack 7 -> Bouton1
- J16: value Jack 8 -> Bouton2
- J2: value Jack 3 -> Jack 2
- J3: value Jack 4 -> Jack 3
- J4: value Jack 5 -> Jack 4
- J5: value Jack 6 -> Jack 5
- J6: value Jack 2 -> Jack 6
- J7: value Jack 0 -> Jack 7
- J8: value Bouton 0 -> Jack 8
- J9: value Bouton 1 -> Jack 9
- R13: value 1.1K -> 10K
- moved R8 38.5 mm to (170.5, 66.8)
- moved J5 38.3 mm to (143.2, 63.2)
- moved R5 35.8 mm to (138.2, 64.2), turned to -90 degrees
- moved J1 35.6 mm to (143.2, 54.5)
- moved U2 35.6 mm to (191.0, 74.0), turned to 90 degrees
- moved J15 34.3 mm to (143.2, 89.8)
- moved J2 32.9 mm to (150.0, 54.5)
- moved R4 32.2 mm to (163.5, 49.8), turned to 90 degrees
- moved R11 31.0 mm to (163.0, 73.0), turned to -90 degrees
- moved R3 30.3 mm to (156.8, 49.8), turned to 90 degrees
- moved J14 30.1 mm to (156.8, 80.8), turned to 0 degrees
- moved J3 30.1 mm to (156.8, 54.5)
- moved R1 30.1 mm to (138.2, 55.5), turned to -90 degrees
- moved J4 29.6 mm to (163.5, 54.5)
- moved R6 29.5 mm to (146.8, 49.8), turned to 90 degrees
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Connections:
- J1 pad 1: B5 -> D2
- J10 pad 1: B2 -> D16
- J10 pad 2: Net-(J10-Pad2) -> Net-(J1-Pad2)
- J11 pad 1: B3 -> D14
- J11 pad 2: Net-(J11-Pad2) -> Net-(J1-Pad2)
- J12 pad 1: B4 -> D15
- J12 pad 2: Net-(J12-Pad2) -> Net-(J1-Pad2)
- J13 pad 1: Net-(J13-Pad1) -> D20
- J13 pad 2: GND -> Net-(J1-Pad2)
- J14 pad 1: A0 -> D21
- J14 pad 2: A1 -> Net-(J1-Pad2)
- J15 pad 1: A2 -> D16
- J15 pad 2: Net-(J15-Pad2) -> Net-(J1-Pad2)
- J16 pad 1: A3 -> D14
- J16 pad 2: Net-(J16-Pad2) -> Net-(J1-Pad2)
- J2 pad 1: B6 -> D3
- J2 pad 2: Net-(J2-Pad2) -> Net-(J1-Pad2)
- J3 pad 1: B7 -> D4
- J3 pad 2: Net-(J3-Pad2) -> Net-(J1-Pad2)
- J4 pad 1: B8 -> D5
- J4 pad 2: Net-(J4-Pad2) -> Net-(J1-Pad2)
- J5 pad 1: B9 -> D6
- J5 pad 2: Net-(J5-Pad2) -> Net-(J1-Pad2)
- J6 pad 1: B10 -> D7
- J6 pad 2: Net-(J6-Pad2) -> Net-(J1-Pad2)
- J7 pad 1: B11 -> D8
- J7 pad 2: Net-(J7-Pad2) -> Net-(J1-Pad2)
- J8 pad 1: B0 -> D9
- J8 pad 2: Net-(J8-Pad2) -> Net-(J1-Pad2)
- J9 pad 1: B1 -> D10
- J9 pad 2: Net-(J9-Pad2) -> Net-(J1-Pad2)
- R1 pad 1: GND -> D2
- R1 pad 2: Net-(J1-Pad2) -> GND
- R10 pad 1: GND -> D16
- R10 pad 2: Net-(J10-Pad2) -> GND
- R11 pad 1: GND -> D14
- R11 pad 2: Net-(J11-Pad2) -> GND
- R12 pad 1: GND -> D15
- R12 pad 2: Net-(J12-Pad2) -> GND
- R13 pad 1: Net-(J14-Pad4) -> D20
- R13 pad 2: Net-(J13-Pad1) -> GND
- R14 pad 1: GND -> D21
- R14 pad 2: Net-(J15-Pad2) -> GND
- R15 pad 1: GND -> D16
- R15 pad 2: Net-(J16-Pad2) -> GND
- R2 pad 1: GND -> D3
- R2 pad 2: Net-(J2-Pad2) -> GND
- R3 pad 1: GND -> D4
- R3 pad 2: Net-(J3-Pad2) -> GND
- R4 pad 1: GND -> D5
- R4 pad 2: Net-(J4-Pad2) -> GND
- R5 pad 1: GND -> D6
- R5 pad 2: Net-(J5-Pad2) -> GND
- R6 pad 1: GND -> D7
- R6 pad 2: Net-(J6-Pad2) -> GND
- R7 pad 1: GND -> D8
- R7 pad 2: Net-(J7-Pad2) -> GND
- R8 pad 1: GND -> D9
- R8 pad 2: Net-(J8-Pad2) -> GND
- R9 pad 1: GND -> D10
- R9 pad 2: Net-(J9-Pad2) -> GND
- U1 pad 15: Net-(J14-Pad4) -> Net-(J1-Pad2)
- U2 pad 10: B5 -> D7
- U2 pad 11: B6 -> D8
- U2 pad 12: B7 -> D9
- U2 pad 13: B8 -> D10
- U2 pad 14: B9 -> D16
- U2 pad 15: B1 -> D14
- U2 pad 16: B0 -> D15
- U2 pad 19: A2 -> D20
- U2 pad 20: A3 -> D21
- U2 pad 21: Net-(J14-Pad4) -> Net-(J1-Pad2)
- U2 pad 5: B11 -> D2
- U2 pad 6: B10 -> D3
- U2 pad 7: B2 -> D4
- U2 pad 8: B3 -> D5
- U2 pad 9: B4 -> D6
Routing:
- net Net-(J1-Pad2): track 0.00 -> 156.0 mm
- net GND: track 0.00 -> 129.1 mm
- net D20: track 0.00 -> 23.5 mm
- net D16: track 0.00 -> 18.3 mm
- net D8: track 0.00 -> 15.7 mm
- net D7: track 0.00 -> 15.3 mm
- net D21: track 0.00 -> 11.2 mm
- net D14: track 0.00 -> 11.0 mm
- net D15: track 0.00 -> 9.75 mm
- net D9: track 0.00 -> 8.62 mm
- net Net-(J20-Pad1): track 0.00 -> 6.75 mm
- net D6: track 0.00 -> 5.00 mm
- net D2: track 0.00 -> 5.00 mm
- net D10: track 0.00 -> 5.00 mm
- net D5: track 0.00 -> 3.75 mm
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Other:
- copper layers 2 -> 4

Commit message: PCB changes
Parts:
- J15: value Bouton1 -> Bouton 1
- J16: value Bouton2 -> Bouton 2
- J17: value Bouton3 -> Bouton 3
- J18: value Bouton4 -> Bouton 4
- J19: value Bouton5 -> Bouton 5
- moved U1 0.50 mm to (114.5, 78.0)
Connections:
- net Net-(J1-Pad2) renamed VCC
Routing:
- net GND: track 129.1 -> 285.2 mm
- net Net-(U1-Pad18): track 0.00 -> 102.8 mm
- net Net-(U1-Pad19): track 0.00 -> 98.8 mm
- net D2: track 5.00 -> 96.7 mm
- net D3: track 3.75 -> 83.6 mm
- net D15: track 9.75 -> 81.2 mm
- net D4: track 3.75 -> 72.2 mm
- net D16: track 18.3 -> 83.8 mm
- net VCC: track 156.0 -> 219.8 mm
- net D6: track 5.00 -> 68.5 mm
- net D14: track 11.0 -> 70.3 mm
- net D5: track 3.75 -> 60.4 mm
- net D7: track 15.3 -> 70.7 mm
- net D20: track 23.5 -> 75.5 mm
- net D10: track 5.00 -> 54.5 mm
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- added copper zone on B.Cu, net GND
- added copper zone on F.Cu, net VCC
Other:
- board outline added: 110 x 60 mm
- board text added: "A0"
- board text added: "A1"
- board text added: "GND"
- board text added: "Mathis Savoie & Jackob Breton"
- board text added: "Projet TSO : Manette adapté Jouer sans limite"

Commit message: quick chanfes
Parts:
- added H1: MountingHole_Pad, MountingHole:MountingHole_3.2mm_M3_Pad_Via, F.Cu at (105.8, 39.8)
- added H2: MountingHole_Pad, MountingHole:MountingHole_3.2mm_M3_Pad_Via, F.Cu at (105.8, 111.2)
- added H3: MountingHole_Pad, MountingHole:MountingHole_3.2mm_M3_Pad_Via, F.Cu at (197.2, 111.2)
- added H4: MountingHole_Pad, MountingHole:MountingHole_3.2mm_M3_Pad_Via, F.Cu at (197.2, 39.8)
- moved U1 4.75 mm to (119.2, 78.0)
- moved U2 3.00 mm to (188.0, 74.0)
Routing:
- net GND: track 285.2 -> 271.9 mm
- net Net-(U1-Pad18): track 102.8 -> 92.6 mm
- net Net-(U1-Pad19): track 98.8 -> 90.9 mm
- net VCC: track 219.8 -> 212.1 mm
- net D2: track 96.7 -> 92.7 mm
- net D3: track 83.6 -> 80.0 mm
- net D4: track 72.2 -> 68.6 mm
- net D5: track 60.4 -> 57.2 mm
- net D16: track 83.8 -> 80.6 mm
- net D10: track 54.5 -> 51.3 mm
- net D9: track 45.5 -> 42.5 mm
- net D8: track 64.0 -> 61.0 mm
- net D7: track 70.7 -> 67.7 mm
- net D6: track 68.5 -> 65.5 mm
- net D20: track 75.5 -> 72.5 mm
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Other:
- board size 110 x 60 mm -> 100 x 80 mm
- board text added: "Finissants Cégep de Sherbrooke 2023"
- board text added: "VCC"
