File: PCB/Manette_JM/Manette_JM.kicad_sch (KiCad schematic)
At the start: 12 parts

Commit message: Schéma électrique et début PCB
Parts:
- removed J?: Joystick 1, symbol Connector:Conn_01x04_Female
- added J13: DEL PWR, Connector_PinHeader_2.54mm:PinHeader_1x02_P2.54mm_Vertical, symbol Connector:Conn_01x02_Female
- added J15: Jack 7, Connector_PinHeader_2.54mm:PinHeader_1x02_P2.54mm_Vertical, symbol Connector:Conn_01x02_Female
- added J16: Jack 8, Connector_PinHeader_2.54mm:PinHeader_1x02_P2.54mm_Vertical, symbol Connector:Conn_01x02_Female
- added J2: Jack 3, Connector_PinHeader_2.54mm:PinHeader_1x02_P2.54mm_Vertical, symbol Connector:Conn_01x02_Female
- added J3: Jack 4, Connector_PinHeader_2.54mm:PinHeader_1x02_P2.54mm_Vertical, symbol Connector:Conn_01x02_Female
- added J4: Jack 5, Connector_PinHeader_2.54mm:PinHeader_1x02_P2.54mm_Vertical, symbol Connector:Conn_01x02_Female
- added J5: Jack 6, Connector_PinHeader_2.54mm:PinHeader_1x02_P2.54mm_Vertical, symbol Connector:Conn_01x02_Female
- added R1, R10, R11, R12, R14, R15, R2, R3, R4, R5, R6, R7, R8, R9: 10K, Resistor_SMD:R_0805_2012Metric_Pad1.20x1.40mm_HandSolder, symbol Device:R
- added R13: 1.1K, Resistor_SMD:R_0805_2012Metric_Pad1.20x1.40mm_HandSolder, symbol Device:R
- J1: renamed from J?; value Bouton 0 -> Jack 1; footprint (none) -> Connector_PinHeader_2.54mm:PinHeader_1x02_P2.54mm_Vertical
- J10: renamed from J?; value Bouton 0 -> Bouton 2; footprint (none) -> Connector_PinHeader_2.54mm:PinHeader_1x02_P2.54mm_Vertical
- J11: renamed from J?; value Bouton 0 -> Bouton 3; footprint (none) -> Connector_PinHeader_2.54mm:PinHeader_1x02_P2.54mm_Vertical
- J12: renamed from J?; value Bouton 0 -> Bouton 4; footprint (none) -> Connector_PinHeader_2.54mm:PinHeader_1x02_P2.54mm_Vertical
- J14: renamed from J?; footprint (none) -> Connector_PinHeader_2.54mm:PinHeader_1x04_P2.54mm_Vertical
- J6: renamed from J?; value Bouton 0 -> Jack 2; footprint (none) -> Connector_PinHeader_2.54mm:PinHeader_1x02_P2.54mm_Vertical
- J7: renamed from J?; value Bouton 0 -> Jack 0; footprint (none) -> Connector_PinHeader_2.54mm:PinHeader_1x02_P2.54mm_Vertical
- J8: renamed from J?; footprint (none) -> Connector_PinHeader_2.54mm:PinHeader_1x02_P2.54mm_Vertical
- J9: renamed from J?; value Bouton 0 -> Bouton 1; footprint (none) -> Connector_PinHeader_2.54mm:PinHeader_1x02_P2.54mm_Vertical
- U1: renamed from U?; footprint (none) -> ESP8266:NodeMCU-LoLinV3
- U2: renamed from U?; footprint (none) -> promicro:ProMicro
Connections:
- net A2: now also J15.1 (Pin_1)
- net A3: now also J16.1 (Pin_1)
- net B0: now also U2.16 (B1); no longer U2.5 (SDA)
- net B1: now also J9.1 (Pin_1), U2.15 (B3); no longer U2.6 (SCL)
- net B10: now also J6.1 (Pin_1), U2.6 (SCL); no longer U2.15 (B3)
- net B11: now also J7.1 (Pin_1), U2.5 (SDA); no longer U2.16 (B1)
- net B2: now also J10.1 (Pin_1)
- net B3: now also J11.1 (Pin_1)
- net B4: now also J12.1 (Pin_1)
- net B5: now also J1.1 (Pin_1)
- net B6: now also J2.1 (Pin_1)
- net B7: now also J3.1 (Pin_1)
- net B8: now also J4.1 (Pin_1)
- net B9: now also J5.1 (Pin_1)
- net GND: now also J13.2 (Pin_2), R1.1, R10.1, R11.1, R12.1, R14.1, R15.1, R2.1, R3.1, R4.1, R5.1, R6.1, R7.1, R8.1, R9.1; no longer J8.2 (Pin_2)
- net at J10.2 (Pin_2): now also R10.2
- net at J9.2 (Pin_2): now also R9.2
- net at J14.4 (Pin_4), U1.15 (VIN), U2.21 (VCC): now also R13.1
- net at J1.2 (Pin_2): now also R1.2
- net at J6.2 (Pin_2): now also R6.2
- net at J12.2 (Pin_2): now also R12.2
- net at J11.2 (Pin_2): now also R11.2
- net at J7.2 (Pin_2): now also R7.2
- new net: J13.1 (Pin_1), R13.2
- new net: J15.2 (Pin_2), R14.2
- new net: J8.2 (Pin_2), R8.2
- new net: J16.2 (Pin_2), R15.2
- new net: J2.2 (Pin_2), R2.2
- new net: J3.2 (Pin_2), R3.2
- new net: J4.2 (Pin_2), R4.2
- new net: J5.2 (Pin_2), R5.2
Other:
- company: (none) -> Cégep de Sherbrooke
- title: (none) -> Manette adaptée 
- moved on the sheet: J1, J10, J11, J12, J6, J7, J8, J9

Commit message: Quick changes
modification code et schéma
Parts:
- removed J10: Bouton 2, Connector_PinHeader_2.54mm:PinHeader_1x02_P2.54mm_Vertical, symbol Connector:Conn_01x02_Female
- removed J11: Bouton 3, Connector_PinHeader_2.54mm:PinHeader_1x02_P2.54mm_Vertical, symbol Connector:Conn_01x02_Female
- removed J12: Bouton 4, Connector_PinHeader_2.54mm:PinHeader_1x02_P2.54mm_Vertical, symbol Connector:Conn_01x02_Female
- removed J8: Bouton 0, Connector_PinHeader_2.54mm:PinHeader_1x02_P2.54mm_Vertical, symbol Connector:Conn_01x02_Female
- removed J9: Bouton 1, Connector_PinHeader_2.54mm:PinHeader_1x02_P2.54mm_Vertical, symbol Connector:Conn_01x02_Female
- added J?: Bouton 1, Connector_PinHeader_2.54mm:PinHeader_1x02_P2.54mm_Vertical, symbol Connector:Conn_01x02_Female
- added J?: Bouton 4, Connector_PinHeader_2.54mm:PinHeader_1x02_P2.54mm_Vertical, symbol Connector:Conn_01x02_Female
- added J?: Jack 12, Connector_PinHeader_2.54mm:PinHeader_1x02_P2.54mm_Vertical, symbol Connector:Conn_01x02_Female
- added J?: Bouton 0, Connector_PinHeader_2.54mm:PinHeader_1x02_P2.54mm_Vertical, symbol Connector:Conn_01x02_Female
- added J?: Jack 10, Connector_PinHeader_2.54mm:PinHeader_1x02_P2.54mm_Vertical, symbol Connector:Conn_01x02_Female
- added J?: Jack 9, Connector_PinHeader_2.54mm:PinHeader_1x02_P2.54mm_Vertical, symbol Connector:Conn_01x02_Female
- added J?: Jack 11, Connector_PinHeader_2.54mm:PinHeader_1x02_P2.54mm_Vertical, symbol Connector:Conn_01x02_Female
- added J?: Bouton 2, Connector_PinHeader_2.54mm:PinHeader_1x02_P2.54mm_Vertical, symbol Connector:Conn_01x02_Female
- added J?: Jack 8, Connector_PinHeader_2.54mm:PinHeader_1x02_P2.54mm_Vertical, symbol Connector:Conn_01x02_Female
- added J?: Bouton 3, Connector_PinHeader_2.54mm:PinHeader_1x02_P2.54mm_Vertical, symbol Connector:Conn_01x02_Female
- added R? (x5): 10K, Resistor_SMD:R_0805_2012Metric_Pad1.20x1.40mm_HandSolder, symbol Device:R
- J15: value Jack 7 -> Jack 13
- J16: value Jack 8 -> Jack 14
- J2: value Jack 3 -> Jack 2
- J3: value Jack 4 -> Jack 3
- J4: value Jack 5 -> Jack 4
- J5: value Jack 6 -> Jack 5
- J6: value Jack 2 -> Jack 6
- J7: value Jack 0 -> Jack 7
Connections:
- net GND: now also R?.1, R?.1, R?.1, R?.1, R?.1
- net at R10.2: now also J?.2 (Pin_2)
- net at R9.2: now also J?.2 (Pin_2)
- net at R8.2: now also J?.2 (Pin_2)
- net at R12.2: now also J?.2 (Pin_2)
- net at R11.2: now also J?.2 (Pin_2)
- net A2 renamed D20
- net D20: now also J?.1 (Pin_1)
- net A3 renamed D21
- net D21: now also J?.1 (Pin_1)
- net B0 renamed D15
- net D15: now also J?.1 (Pin_1)
- net B1 renamed D14
- net D14: now also J?.1 (Pin_1)
- net B10 renamed D3
- net D3: now also J2.1 (Pin_1); no longer J6.1 (Pin_1)
- net B11 renamed D2
- net D2: now also J1.1 (Pin_1); no longer J7.1 (Pin_1)
- net B2 renamed D4
- net D4: now also J3.1 (Pin_1)
- net B3 renamed D5
- net D5: now also J4.1 (Pin_1)
- net B4 renamed D6
- net D6: now also J5.1 (Pin_1)
- net B5 renamed D7
- net D7: now also J6.1 (Pin_1); no longer J1.1 (Pin_1)
- net B6 renamed D8
- net D8: now also J7.1 (Pin_1); no longer J2.1 (Pin_1)
- net B7 renamed D9
- net D9: now also J?.1 (Pin_1); no longer J3.1 (Pin_1)
- net B8 renamed D10
- net D10: now also J?.1 (Pin_1); no longer J4.1 (Pin_1)
- net B9 renamed D16
- net D16: now also J?.1 (Pin_1), J?.1 (Pin_1); no longer J5.1 (Pin_1)
- new net: J?.2 (Pin_2), R?.2 (x5)
- new net D17: J?.1 (Pin_1)
- new net D18: J?.1 (Pin_1)
Other:
- moved on the sheet: J1, J13, J14, J15, J16, J2, J3, J4, J5, J6, J7, R1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

Commit message: PCB upgrade
Parts:
- removed J?: Bouton 1, Connector_PinHeader_2.54mm:PinHeader_1x02_P2.54mm_Vertical, symbol Connector:Conn_01x02_Female
- removed J?: Bouton 4, Connector_PinHeader_2.54mm:PinHeader_1x02_P2.54mm_Vertical, symbol Connector:Conn_01x02_Female
- removed J?: Jack 12, Connector_PinHeader_2.54mm:PinHeader_1x02_P2.54mm_Vertical, symbol Connector:Conn_01x02_Female
- removed J?: Bouton 0, Connector_PinHeader_2.54mm:PinHeader_1x02_P2.54mm_Vertical, symbol Connector:Conn_01x02_Female
- removed J?: Jack 10, Connector_PinHeader_2.54mm:PinHeader_1x02_P2.54mm_Vertical, symbol Connector:Conn_01x02_Female
- removed J?: Jack 9, Connector_PinHeader_2.54mm:PinHeader_1x02_P2.54mm_Vertical, symbol Connector:Conn_01x02_Female
- removed J?: Jack 11, Connector_PinHeader_2.54mm:PinHeader_1x02_P2.54mm_Vertical, symbol Connector:Conn_01x02_Female
- removed J?: Bouton 2, Connector_PinHeader_2.54mm:PinHeader_1x02_P2.54mm_Vertical, symbol Connector:Conn_01x02_Female
- removed J?: Jack 8, Connector_PinHeader_2.54mm:PinHeader_1x02_P2.54mm_Vertical, symbol Connector:Conn_01x02_Female
- removed J?: Bouton 3, Connector_PinHeader_2.54mm:PinHeader_1x02_P2.54mm_Vertical, symbol Connector:Conn_01x02_Female
- removed R? (x5): 10K, Resistor_SMD:R_0805_2012Metric_Pad1.20x1.40mm_HandSolder, symbol Device:R
- added J10: Jack 10, Connector_PinHeader_2.54mm:PinHeader_1x02_P2.54mm_Vertical, symbol Connector:Conn_01x02_Female
- added J11: Jack 11, Connector_PinHeader_2.54mm:PinHeader_1x02_P2.54mm_Vertical, symbol Connector:Conn_01x02_Female
- added J12: Jack 12, Connector_PinHeader_2.54mm:PinHeader_1x02_P2.54mm_Vertical, symbol Connector:Conn_01x02_Female
- added J13: Jack 13, Connector_PinHeader_2.54mm:PinHeader_1x02_P2.54mm_Vertical, symbol Connector:Conn_01x02_Female
- added J14: Jack 14, Connector_PinHeader_2.54mm:PinHeader_1x02_P2.54mm_Vertical, symbol Connector:Conn_01x02_Female
- added J17: Bouton 3, Connector_PinHeader_2.54mm:PinHeader_1x02_P2.54mm_Vertical, symbol Connector:Conn_01x02_Female
- added J18: Bouton 4, Connector_PinHeader_2.54mm:PinHeader_1x02_P2.54mm_Vertical, symbol Connector:Conn_01x02_Female
- added J19: Bouton 5, Connector_PinHeader_2.54mm:PinHeader_1x02_P2.54mm_Vertical, symbol Connector:Conn_01x02_Female
- added J8: Jack 8, Connector_PinHeader_2.54mm:PinHeader_1x02_P2.54mm_Vertical, symbol Connector:Conn_01x02_Female
- added J9: Jack 9, Connector_PinHeader_2.54mm:PinHeader_1x02_P2.54mm_Vertical, symbol Connector:Conn_01x02_Female
- added R13, R16, R17, R18, R19: 10K, Resistor_SMD:R_0805_2012Metric_Pad1.20x1.40mm_HandSolder, symbol Device:R
- J15: value Jack 13 -> Bouton 1
- J16: value Jack 14 -> Bouton 2
- renumbered J13 to J20, J14 to J21, R13 to R20
Connections:
- net D10: now also R9.1, J9.1 (Pin_1)
- net D14: now also J16.1 (Pin_1), R11.1, J11.1 (Pin_1), R16.1
- net D15: now also R12.1, J12.1 (Pin_1), J17.1 (Pin_1), R17.1
- net D16: now also J15.1 (Pin_1), R10.1, R15.1, J10.1 (Pin_1)
- net D2: now also R1.1
- net D20: now also J13.1 (Pin_1), J18.1 (Pin_1), R13.1, R18.1; no longer J15.1 (Pin_1)
- net D21: now also R14.1, J14.1 (Pin_1), J19.1 (Pin_1), R19.1; no longer J16.1 (Pin_1)
- net D3: now also R2.1
- net D4: now also R3.1
- net D5: now also R4.1
- net D6: now also R5.1
- net D7: now also R6.1
- net D8: now also R7.1
- net D9: now also R8.1, J8.1 (Pin_1)
- net GND: now also R1.2, R10.2, R11.2, R12.2, R14.2, R15.2, R2.2, R3.2, R4.2, R5.2, R6.2, R7.2, R8.2, R9.2, R13.2, R16.2, R17.2, R18.2, R19.2; no longer R1.1, R10.1, R11.1, R12.1, R14.1, R15.1, R2.1, R3.1, R4.1, R5.1, R6.1, R7.1, R8.1, R9.1
- net at J21.4 (Pin_4), R20.1, U1.15 (VIN)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: now also J1.2 (Pin_2), J15.2 (Pin_2), J16.2 (Pin_2), J2.2 (Pin_2), J3.2 (Pin_2), J4.2 (Pin_2), J5.2 (Pin_2), J6.2 (Pin_2), J7.2 (Pin_2), J10.2 (Pin_2), J11.2 (Pin_2), J12.2 (Pin_2), J13.2 (Pin_2), J14.2 (Pin_2), J17.2 (Pin_2), J18.2 (Pin_2), J19.2 (Pin_2), J8.2 (Pin_2), J9.2 (Pin_2)
- no-connect marks 0 -> 25
Other:
- moved on the sheet: J1, J2, J3, J4, J5, J6, J7, R1, R2, R3, R4, R5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

Commit message: PCB changes
Connections:
- net VCC: now reaches J1.2 (Pin_2), J10.2 (Pin_2), J11.2 (Pin_2), J12.2 (Pin_2), J13.2 (Pin_2), J14.2 (Pin_2), J15.2 (Pin_2), J16.2 (Pin_2), J17.2 (Pin_2), J18.2 (Pin_2), J19.2 (Pin_2), J2.2 (Pin_2), J21.4 (Pin_4), J3.2 (Pin_2), J4.2 (Pin_2), J5.2 (Pin_2), J6.2 (Pin_2), J7.2 (Pin_2), J8.2 (Pin_2), J9.2 (Pin_2), R20.1, U1.15 (VIN), U2.21 (VCC)
Changed lines of the file:
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@@
   (junction (at 68.453 111.633) (diameter 0) (color 0 0 0 0)
+  )
+  (junction (at 189.611 51.943) (diameter 0) (color 0 0 0 0)
   )
   (junction (at 55.372 77.343) (diameter 0) (color 0 0 0 0)
@@
     (stroke (width 0) (type default) (color 0 0 0 0))
   )
-  (wire (pts (xy 179.197 51.943) (xy 200.152 51.943))
+  (wire (pts (xy 179.197 51.943) (xy 189.611 51.943))
     (stroke (width 0) (type default) (color 0 0 0 0))
   )
@@
   )
   (wire (pts (xy 85.09 146.558) (xy 85.09 158.623))
+    (stroke (width 0) (type default) (color 0 0 0 0))
+  )
+  (wire (pts (xy 189.611 51.943) (xy 200.152 51.943))
     (stroke (width 0) (type default) (color 0 0 0 0))
   )
@@
     (pin "1")
     (pin "2")
+  )
+  (symbol (lib_id "power:VCC") (at 189.611 51.943 0) (unit 1)
+    (in_bom yes) (on_board yes) (fields_autoplaced)
+    (property "Reference" "#PWR0101" (id 0) (at 189.611 55.753 0)
+      (effects (font (size 1.27 1.27)) hide)
+    )
+    (property "Value" "VCC" (id 1) (at 189.611 48.3385 0))
+    (property "Footprint" "" (id 2) (at 189.611 51.943 0)
+      (effects (font (size 1.27 1.27)) hide)
+    )
+    (property "Datasheet" "" (id 3) (at 189.611 51.943 0)
+      (effects (font (size 1.27 1.27)) hide)
+    )
+    (pin "1")
   )
   (symbol (lib_id "Connector:Conn_01x02_Female") (at 144.653 149.987 0) (unit 1)
@@
       (reference "#PWR09") (unit 1) (value "GND") (footprint "")
     )
+    (path "/082ecb16-bdc7-404f-9607-610400050981"
+      (reference "#PWR0101") (unit 1) (value "VCC") (footprint "")
+    )
     (path "/6bd69486-05a5-4980-a8b7-59af08aa7936"

Commit message: quick chanfes
Parts:
- added H1, H2, H3, H4: MountingHole_Pad, MountingHole:MountingHole_3.2mm_M3_Pad_Via, symbol Mechanical:MountingHole_Pad
Connections:
- no-connect marks 25 -> 29
Changed lines of the file:
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@@
   (junction (at 95.123 152.527) (diameter 0) (color 0 0 0 0)
   )
+  (no_connect (at 201.803 116.967))
+  (no_connect (at 225.933 117.221))
+  (no_connect (at 225.933 131.064))
+  (no_connect (at 201.803 131.191))
   (no_connect (at 105.537 62.103))
   (no_connect (at 105.537 79.883))
@@
   (symbol (lib_id "power:VCC") (at 189.611 51.943 0) (unit 1)
     (in_bom yes) (on_board yes) (fields_autoplaced)
-    (property "Reference" "#PWR0101" (id 0) (at 189.611 55.753 0)
+    (property "Reference" "#PWR09" (id 0) (at 189.611 55.753 0)
       (effects (font (size 1.27 1.27)) hide)
     )
@@
   (symbol (lib_id "power:PWR_FLAG") (at 200.152 46.863 0) (unit 1)
     (in_bom yes) (on_board yes)
-    (property "Reference" "#FLG0101" (id 0) (at 200.152 44.958 0)
+    (property "Reference" "#FLG01" (id 0) (at 200.152 44.958 0)
       (effects (font (size 1.27 1.27)) hide)
     )
@@
   (symbol (lib_id "power:PWR_FLAG") (at 200.152 51.943 0) (unit 1)
     (in_bom yes) (on_board yes)
-    (property "Reference" "#FLG0102" (id 0) (at 200.152 50.038 0)
+    (property "Reference" "#FLG02" (id 0) (at 200.152 50.038 0)
       (effects (font (size 1.27 1.27)) hide)
     )
@@
     )
     (property "Datasheet" "~" (id 3) (at 200.152 51.943 0)
+      (effects (font (size 1.27 1.27)) hide)
+    )
+    (pin "1")
+  )
+  (symbol (lib_id "Mechanical:MountingHole_Pad") (at 225.933 128.524 0) (unit 1)
+    (in_bom yes) (on_board yes) (fields_autoplaced)
+    (property "Reference" "H4" (id 0) (at 228.473 126.3455 0)
+      (effects (font (size 1.27 1.27)) (justify left))
+    )
+    (property "Value" "MountingHole_Pad" (id 1) (at 228.473 129.1206 0)
+      (effects (font (size 1.27 1.27)) (justify left))
+    )
+    (property "Footprint" "MountingHole:MountingHole_3.2mm_M3_Pad_Via" (id 2) (at 225.933 128.524 0)
+      (effects (font (size 1.27 1.27)) hide)
+    )
+    (property "Datasheet" "~" (id 3) (at 225.933 128.524 0)
       (effects (font (size 1.27 1.27)) hide)
     )
@@
     (pin "2")
   )
+  (symbol (lib_id "Mechanical:MountingHole_Pad") (at 201.803 114.427 0) (unit 1)
+    (in_bom yes) (on_board yes) (fields_autoplaced)
+    (property "Reference" "H1" (id 0) (at 204.343 112.2485 0)
+      (effects (font (size 1.27 1.27)) (justify left))
+    )
+    (property "Value" "MountingHole_Pad" (id 1) (at 204.343 115.0236 0)
+      (effects (font (size 1.27 1.27)) (justify left))
+    )
+    (property "Footprint" "MountingHole:MountingHole_3.2mm_M3_Pad_Via" (id 2) (at 201.803 114.427 0)
+      (effects (font (size 1.27 1.27)) hide)
+    )
+    (property "Datasheet" "~" (id 3) (at 201.803 114.427 0)
+      (effects (font (size 1.27 1.27)) hide)
+    )
+    (pin "1")
+  )
   (symbol (lib_id "power:GND") (at 109.347 59.563 0) (unit 1)
     (in_bom yes) (on_board yes) (fields_autoplaced)
@@
     )
     (property "Datasheet" "" (id 3) (at 109.347 77.343 0)
+      (effects (font (size 1.27 1.27)) hide)
+    )
+    (pin "1")
+  )
+  (symbol (lib_id "Mechanical:MountingHole_Pad") (at 201.803 128.651 0) (unit 1)
+    (in_bom yes) (on_board yes) (fields_autoplaced)
+    (property "Reference" "H2" (id 0) (at 204.343 126.4725 0)
+      (effects (font (size 1.27 1.27)) (justify left))
+    )
+    (property "Value" "MountingHole_Pad" (id 1) (at 204.343 129.2476 0)
+      (effects (font (size 1.27 1.27)) (justify left))
+    )
+    (property "Footprint" "MountingHole:MountingHole_3.2mm_M3_Pad_Via" (id 2) (at 201.803 128.651 0)
+      (effects (font (size 1.27 1.27)) hide)
+    )
+    (property "Datasheet" "~" (id 3) (at 201.803 128.651 0)
       (effects (font (size 1.27 1.27)) hide)
     )
@@
   (symbol (lib_id "power:GND") (at 218.567 83.058 0) (unit 1)
     (in_bom yes) (on_board yes) (fields_autoplaced)
-    (property "Reference" "#PWR09" (id 0) (at 218.567 89.408 0)
+    (property "Reference" "#PWR010" (id 0) (at 218.567 89.408 0)
       (effects (font (size 1.27 1.27)) hide)
     )
@@
     (pin "2")
   )
+  (symbol (lib_id "Mechanical:MountingHole_Pad") (at 225.933 114.681 0) (unit 1)
+    (in_bom yes) (on_board yes) (fields_autoplaced)
+    (property "Reference" "H3" (id 0) (at 228.473 112.5025 0)
+      (effects (font (size 1.27 1.27)) (justify left))
+    )
+    (property "Value" "MountingHole_Pad" (id 1) (at 228.473 115.2776 0)
+      (effects (font (size 1.27 1.27)) (justify left))
+    )
+    (property "Footprint" "MountingHole:MountingHole_3.2mm_M3_Pad_Via" (id 2) (at 225.933 114.681 0)
+      (effects (font (size 1.27 1.27)) hide)
+    )
+    (property "Datasheet" "~" (id 3) (at 225.933 114.681 0)
+      (effects (font (size 1.27 1.27)) hide)
+    )
+    (pin "1")
+  )
   (symbol (lib_id "Device:R") (at 76.708 146.558 90) (unit 1)
     (in_bom yes) (on_board yes)
@@
   (symbol_instances
     (path "/2aea3883-9bba-4418-9eac-85986d3d4e6d"
-      (reference "#FLG0101") (unit 1) (value "PWR_FLAG") (footprint "")
+      (reference "#FLG01") (unit 1) (value "PWR_FLAG") (footprint "")
     )
     (path "/2bfe5755-98c1-411c-947a-07ba5e9332a3"
-      (reference "#FLG0102") (unit 1) (value "PWR_FLAG") (footprint "")
+      (reference "#FLG02") (unit 1) (value "PWR_FLAG") (footprint "")
     )
     (path "/d122d081-7fdf-4b0c-b695-88d167a2f3da"
@@
       (reference "#PWR08") (unit 1) (value "GND") (footprint "")
     )
+    (path "/082ecb16-bdc7-404f-9607-610400050981"
+      (reference "#PWR09") (unit 1) (value "VCC") (footprint "")
+    )
     (path "/d153de0a-2194-4c66-b9b0-b9eb50365793"
-      (reference "#PWR09") (unit 1) (value "GND") (footprint "")
-    )
-    (path "/082ecb16-bdc7-404f-9607-610400050981"
-      (reference "#PWR0101") (unit 1) (value "VCC") (footprint "")
+      (reference "#PWR010") (unit 1) (value "GND") (footprint "")
+    )
+    (path "/391e77f9-45fd-4544-9a96-6b9be0f3494b"
+      (reference "H1") (unit 1) (value "MountingHole_Pad") (footprint "MountingHole:MountingHole_3.2mm_M3_Pad_Via")
+    )
+    (path "/7f47ecb6-4909-48a6-b1c5-f4bda50df92d"
+      (reference "H2") (unit 1) (value "MountingHole_Pad") (footprint "MountingHole:MountingHole_3.2mm_M3_Pad_Via")
+    )
+    (path "/f9068831-8f5b-4b4f-886a-9c4e538eb3c4"
+      (reference "H3") (unit 1) (value "MountingHole_Pad") (footprint "MountingHole:MountingHole_3.2mm_M3_Pad_Via")
+    )
+    (path "/2e74c5cf-df21-4ecb-90c2-e2781152c95b"
+      (reference "H4") (unit 1) (value "MountingHole_Pad") (footprint "MountingHole:MountingHole_3.2mm_M3_Pad_Via")
     )
     (path "/6bd69486-05a5-4980-a8b7-59af08aa7936"
